File: elektroniikka/control_board.kicad_sch (KiCad schematic)
At the start: 5 parts, among them K1 Relay_SPST-NO, Q1 IRFZ44N, U1 L7805CV

Commit message: timesorting works
Parts:
- added D1, D2, D3, D4: LED, symbol Device:LED
- added R1, R2, R3, R4: 68, symbol Device:R
- added R5, R6, R7, R8: R, symbol Device:R
- added SW1, SW2, SW3, SW4: mom dip, symbol Switch:SW_DIP_x01
Connections:
- net GND: now also R1.2, R2.2, R3.2, R4.2, SW1.2, SW2.2, SW3.2, SW4.2
- new net: D3.1 (K), R3.1
- new net: R6.2, SW2.1
- new net: R5.2, SW1.1
- new net: D1.1 (K), R1.1
- new net: D2.1 (K), R2.1
- new net: R8.2, SW4.1
- new net: R7.2, SW3.1
- new net: D4.1 (K), R4.1
- new net +3.3V: R5.1, R6.1, R7.1, R8.1
Other:
- note added: "State indicator leds, to outputs of esp"
- note added: "dip switches for conrol, to inputs of esp"

Commit message: timezone stuff, nettiin harvemmin
Other:
- note added: "IF using 24 volt suply this will heat up to much, use switching regulator instead"
Changed lines of the file:
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@@
+		)
+	)
+	(text "IF using 24 volt suply this will heat up to much, use  switching regulator instead"
+		(exclude_from_sim no)
+		(at 47.244 70.612 0)
+		(effects
+			(font
+				(size 1.27 1.27)
+			)
 		)
 	)
